File: MasterBoard.kicad_pcb (KiCad board)
At the start: 2 copper layers, 6 parts, among them U1 STM32F103ZETx, U2 DS18B20, U3 DS18B20, U4 W5500, U5 DS18B20, U6 DS18B20

Commit message: kicad final
Parts:
- removed the U5 at (58.9, 49.1)
- added D1: 1N5822, Diode_THT:D_DO-201AD_P15.24mm_Horizontal, F.Cu at (170.7, 91.0)
- added D2: SMAJ5.0A, Diode_THT:D_DO-201AD_P15.24mm_Horizontal, F.Cu at (141.1, 55.5)
- added D4: 1N5822, Diode_THT:D_DO-201AD_P15.24mm_Horizontal, F.Cu at (130.2, 80.6)
- added IC1: W5500, WIZW5500:QFP50P900X900X160-48N, F.Cu at (131.8, 91.7)
- added J9: HR911105A, HR911105A:HR911105A, F.Cu at (107.2, 87.5)
- added U10: AMS1117-3.3, Package_TO_SOT_SMD:SOT-223-3_TabPin2, F.Cu at (134.3, 57.0)
- added U2: STM32F103ZETx, Package_QFP:LQFP-144_20x20mm_P0.5mm, F.Cu at (115.3, 68.8)
- added U3: STM32F103ZETx, Package_QFP:LQFP-144_20x20mm_P0.5mm, F.Cu at (118.9, 40.6)
- added U8: DS18B20, Package_TO_SOT_THT:TO-92_Inline, F.Cu at (145.6, 68.4)
- added U9: LM2596S-5.0, Package_TO_SOT_SMD:TO-263-5_TabPin3, F.Cu at (164.2, 63.6)
- added XATL2: 32.768kHz, CFS_Crystal_32kHz:CFS20632768DZFB, F.Cu at (142.8, 73.5)
- U4: value W5500 -> STM32F103ZETx; footprint Package_QFP:LQFP-48_7x7mm_P0.5mm -> Package_QFP:LQFP-144_20x20mm_P0.5mm
- moved U1 118.3 mm to (154.1, 85.8)
- moved U4 97.4 mm to (159.8, 40.2)
- moved U5 81.2 mm to (136.0, 68.8)
- moved U7 80.2 mm to (136.1, 81.1)
- moved U6 79.0 mm to (136.4, 75.1)
- renumbered U2 to U5, U3 to U6, U6 to U7
Connections:
- net Net-(U1-Pad1) renamed Bak_SPI_MISO
- net Net-(U1-Pad101) renamed USART1_TX
- net Net-(U1-Pad102) renamed USART1_RX
- net Net-(U1-Pad105) renamed JTMS\SWDIO
- net Net-(U1-Pad107) renamed VSS8
- net Net-(U1-Pad108) renamed VDD8
- net Net-(U1-Pad109) renamed JTCK\SWCLK
- net Net-(U1-Pad110) renamed JTDI
- net Net-(U1-Pad120) renamed VSS9
- net Net-(U1-Pad121) renamed VDD9
- net Net-(U1-Pad130) renamed VSS10
- net Net-(U1-Pad131) renamed VDD10
- net Net-(U1-Pad142) renamed Bak_SPI_SCK
- net Net-(U1-Pad143) renamed VSS11
- net Net-(U1-Pad144) renamed VDD11
- net Net-(U1-Pad16) renamed VSS1
- net Net-(U1-Pad17) renamed VDD1
- net Net-(U1-Pad2) renamed Bak_SPI_MOSI
- net Net-(U1-Pad30) renamed VSSA
- net Net-(U1-Pad31) renamed VREF-
- net Net-(U1-Pad32) renamed VREF+
- net Net-(U1-Pad33) renamed VDDA
- net Net-(U1-Pad38) renamed VSS2
- net Net-(U1-Pad39) renamed VDD2
- net Net-(U1-Pad48) renamed BOOT1
- net Net-(U1-Pad51) renamed VSS3
- net Net-(U1-Pad52) renamed VDD3
- net Net-(U1-Pad6) renamed VBAT
- net Net-(U1-Pad61) renamed VSS4
- net Net-(U1-Pad62) renamed VDD4
- net Net-(U1-Pad71) renamed VSS5
- net Net-(U1-Pad72) renamed VDD5
- net Net-(U1-Pad83) renamed VSS6
- net Net-(U1-Pad84) renamed VDD6
- net Net-(U1-Pad94) renamed VSS7
- net Net-(U1-Pad95) renamed VDD7
- net Net-(U4-Pad18) renamed S4_ADC14
- net Net-(U4-Pad20) renamed S4_ADC16
- net Net-(U4-Pad22) renamed S4_ADC18
- net Net-(U4-Pad26) renamed S4_ADC08
- net Net-(U4-Pad27) renamed S4_ADC09
- net Net-(U4-Pad28) renamed S4_ADC10
- net Net-(U4-Pad29) renamed S4_ADC11
- net Net-(U4-Pad30) renamed S4_VSSA
- net Net-(U4-Pad31) renamed S4_VREF-
- net Net-(U4-Pad32) renamed S4_VREF+
- net Net-(U4-Pad33) renamed S4_VDDA
- net Net-(U4-Pad34) renamed S4_ADC01
- net Net-(U4-Pad35) renamed S4_ADC02
- net Net-(U4-Pad36) renamed S4_ADC03
- net Net-(U4-Pad37) renamed S4_ADC04
- net Net-(U4-Pad38) renamed S4_VSS2
- net Net-(U4-Pad39) renamed S4_VDD2
- net Net-(U4-Pad40) renamed S4_ADC05
- net Net-(U4-Pad44) renamed S4_ADC12
- net Net-(U4-Pad45) renamed S4_ADC13
- net Net-(U4-Pad46) renamed S4_ADC06
- net Net-(U4-Pad47) renamed S4_ADC07
- net PB3 renamed JTDO\SWO
- net PB4 renamed JTRST
- net PB5 renamed Net-(U1-Pad135)
- U1 pad 11: Net-(U1-Pad11) -> DQ1
- U1 pad 12: Net-(U1-Pad12) -> DQ2
- U1 pad 13: Net-(U1-Pad13) -> DQ3
- U1 pad 14: Net-(U1-Pad14) -> DQ4
- U1 pad 3: Net-(U1-Pad3) -> SW_RESET
- U1 pad 41: Net-(U1-Pad41) -> M_SPI1_SCK
- U1 pad 42: Net-(U1-Pad42) -> M_SPI1_MISO
- U1 pad 43: Net-(U1-Pad43) -> M_SPI1_MOSI
- U1 pad 73: Net-(U1-Pad73) -> W5500_SCS
- U1 pad 74: PB13 -> W5500_SPI2_SCLK
- U1 pad 75: PB14 -> W5500_SPI2_MISO
- U1 pad 76: PB15 -> W5500_SPI2_MOSI
- U1 pad 8: Net-(U1-Pad8) -> OSC32_IN
- U1 pad 9: Net-(U1-Pad9) -> OSC32_OUT
- U1 pad 96: Net-(U1-Pad96) -> W5500_INT
- U1 pad 97: Net-(U1-Pad97) -> W5500_RST
- U4 pad 15: Net-(U4-Pad11) -> Net-(U4-Pad15)
- U4 pad 16: Net-(U4-Pad14) -> S4_VSS1
- U4 pad 17: Net-(U4-Pad11) -> S4_VDD1
- U4 pad 19: Net-(U4-Pad14) -> S4_ADC15
- U4 pad 21: Net-(U4-Pad11) -> S4_ADC17
- U4 pad 3: Net-(U4-Pad14) -> SW_RESET
- U4 pad 4: Net-(U4-Pad11) -> Net-(U4-Pad4)
- U4 pad 41: Net-(U4-Pad41) -> S2_S4_SPI3_SCLK
- U4 pad 42: Net-(U4-Pad42) -> S2_S4_SPI3_MISO
- U4 pad 43: Net-(U4-Pad43) -> S2_S4_SPI3_MOSI
- U4 pad 48: Net-(U4-Pad14) -> Net-(R40-Pad1)
- U4 pad 8: Net-(U4-Pad11) -> Net-(U4-Pad8)
- U4 pad 9: Net-(U4-Pad14) -> Net-(U4-Pad9)
- U5 pad 1: Net-(U2-Pad1) -> GND
- U5 pad 2: Net-(U2-Pad2) -> DQ1
- U5 pad 3: Net-(U2-Pad3) -> +5V
- U6 pad 1: Net-(U3-Pad1) -> GND
- U6 pad 2: Net-(U3-Pad2) -> DQ2
- U6 pad 3: Net-(U3-Pad3) -> +5V
- U7 pad 1: Net-(U6-Pad1) -> GND
- U7 pad 2: Net-(U6-Pad2) -> DQ3
- U7 pad 3: Net-(U6-Pad3) -> +5V
Routing:
- net GND: track 0.00 -> 191.6 mm, vias 0 -> 1
- net SW_RESET: track 0.00 -> 129.7 mm
- net +3V3: track 0.00 -> 70.2 mm, vias 0 -> 2
- net +5V: track 0.00 -> 58.8 mm
- net M_SPI1_MISO: track 0.00 -> 57.8 mm
- net M_SPI1_SCK: track 0.00 -> 49.1 mm
- net M_SPI1_MOSI: track 0.00 -> 49.1 mm
- net S2_S4_SPI3_MOSI: track 0.00 -> 47.9 mm
- net S2_S4_SPI3_MISO: track 0.00 -> 47.0 mm
- net S2_S4_SPI3_SCLK: track 0.00 -> 45.0 mm
- net S2_S3_SPI2_SCLK: track 0.00 -> 39.3 mm
- net S2_S3_SPI2_MOSI: track 0.00 -> 38.7 mm
- net Net-(C19-Pad1): track 0.00 -> 37.4 mm
- net W5500_SPI2_MISO: track 0.00 -> 37.1 mm
- net W5500_SPI2_SCLK: track 0.00 -> 37.0 mm
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Other:
- board outline added: 75 x 75 mm
