File: MasterBoard.sch (KiCad schematic (older format))
At the start: 75 parts, among them J1 Conn_01x02, J1 Header 10X2, J2 Header 01x06, J2 Jack-DC, J3 +5V, J6 USB_B_Micro, SW1 RESET, SW2 SW_DIP_x01, SW2 SW_DPDT_x2, U1 STM32F103ZETx, U2 DS18B20, U2 LM2596S-5.0, U3 AMS1117-3.3, U3 DS18B20, U4 CH340G, U4 DS18B20, U5 DS18B20, U6 W5500, Y3 12MHz

Commit message: kicad final
Parts:
- removed 1M1: R, symbol Device:R
- removed C27: 10uF, symbol Device:CP
- removed D5: 1N4148, Diode_THT:D_DO-35_SOD27_P7.62mm_Horizontal, symbol Diode:1N4148
- removed F1: Fuse, symbol Device:Fuse
- removed J6: USB_B_Micro, symbol Connector:USB_B_Micro
- removed JP1, JP2: Jumper_NO_Small, symbol Device:Jumper_NO_Small
- removed R10: 100k, symbol Device:R
- removed SW2: SW_DPDT_x2, symbol Switch:SW_DPDT_x2
- removed SW?: SW_DIP_x12, symbol Switch:SW_DIP_x12
- removed U4: CH340G, Package_SO:SOIC-16_3.9x9.9mm_P1.27mm, symbol Interface_USB:CH340G
- removed U6: W5500, Package_QFP:LQFP-48_7x7mm_P0.5mm, symbol Interface_Ethernet:W5500
- removed Y3: 12MHz, symbol Device:Crystal
- added C27, C33, C34, C35, C36, C37, C38, C39, C40, C41, C42, C43, C44, C45, C46, C47, C48, C49, C50, C51, C52, C53, C54, C55, C56, C57, C58, C63: 104, symbol Device:C
- added C59: 22nF, symbol Device:C
- added C60, C62: 6.8nF, symbol Device:C
- added C61: 0.01uF, symbol Device:C
- added C64: 4.7uF, symbol Device:C
- added C65: 10nF, symbol Device:C
- added C66, C67: 18pF, symbol Device:C
- added C68, C69, C70, C71, C72, C73: 30pF, symbol Device:CP1
- added IC1: W5500, QFP50P900X900X160-48N, symbol WIZW5500:W5500
- added J21, J31, J41: Conn_02x09_Odd_Even, symbol Connector_Generic:Conn_02x09_Odd_Even
- added J22: Header 01x06, symbol Connector_Generic:Conn_01x06
- added J32, J33, J42, J43, J5: Conn_01x03, symbol Connector_Generic:Conn_01x03
- added J4: Conn_01x04, symbol Connector_Generic:Conn_01x04
- added J9: HR911105A, HR911105A, symbol HR911105A:HR911105A
- added R13, R14: 51R, symbol Device:R
- added R15: 10R, symbol Device:R
- added R16, R17: 1K, symbol Device:R
- added R18, R19: 82R, symbol Device:R
- added R20: 12.4K, symbol Device:R
- added R21, R22, R23, R24, R25, R26, R27, R28, R29: 10K, symbol Device:R
- added R30: 1M, symbol Device:R
- added R31, R32, R33, R34, R35, R36, R37, R38, R39, R40: 10k, symbol Device:R
- added R9: 100K, symbol Device:R
- added SW2: SW_Push, symbol Switch:SW_Push
- added SW4, SW5, SW6: SW_Push_Dual, symbol Switch:SW_Push_Dual
- added U2, U3, U4: STM32F103ZETx, Package_QFP:LQFP-144_20x20mm_P0.5mm, symbol MCU_ST_STM32F1:STM32F103ZETx
- added XATL3: 25MHz, symbol Device:Crystal
- added XATL4, XATL5, XATL6: 8MHz, symbol Device:Crystal
- C28, C30: value 22pF -> 104
- C31: value C -> 104
- C32: value 22uF -> 104
- gave numbers to parts that had none: 2
- renumbered C15 to C13, C16 to C14, C17 to C15, C18 to C16, J2 to J6, J1 to J7, J3 to J8, R5 to R12, SW2 to SW3, U3 to U10, U2 to U5, U3 to U6, U4 to U7, U5 to U8, U2 to U9, XTAL2 to XATL2
Connections:
- net labels added: ACTLED, Bak_SPI_MISO, Bak_SPI_MOSI, Bak_SPI_SCK, LINKLED, M_SPI1_MISO, M_SPI1_MOSI, M_SPI1_SCK, RCT, RXN, RXNNET, RXP, RXPNET, S2_ADC01, S2_ADC02, S2_ADC03, S2_ADC04, S2_ADC05, S2_ADC06, S2_ADC07, S2_ADC08, S2_ADC09, S2_ADC10, S2_ADC11, S2_ADC12, S2_ADC13, S2_ADC14, S2_ADC15, S2_ADC16, S2_ADC17, S2_ADC18, S2_S3_SPI2_MISO, S2_S3_SPI2_MOSI, S2_S3_SPI2_SCLK, S2_S4_SPI3_MISO, S2_S4_SPI3_MOSI, S2_S4_SPI3_SCLK, S2_SWCLK, S2_SWDIO, S2_VDD1, S2_VDD10, S2_VDD11, S2_VDD2, S2_VDD3, S2_VDD4, S2_VDD5, S2_VDD6, S2_VDD7, S2_VDD8, S2_VDD9, S2_VDDA, S2_VREF+, S2_VREF-, S2_VSS1, S2_VSS10, S2_VSS11, S2_VSS2, S2_VSS3, S2_VSS4, S2_VSS5, S2_VSS6, S2_VSS7, S2_VSS8, S2_VSS9, S2_VSSA, S3_ADC01, S3_ADC02, S3_ADC03, S3_ADC04, S3_ADC05, S3_ADC06, S3_ADC07, S3_ADC08, S3_ADC09, S3_ADC10, S3_ADC11, S3_ADC12, S3_ADC13, S3_ADC14, S3_ADC15, S3_ADC16, S3_ADC17, S3_ADC18, S3_SPI2_MISO, S3_SPI2_MOSI, S3_SPI2_SCLK, S3_SPI3_MISO, S3_SPI3_MOSI, S3_SPI3_SCK, S3_SWCLK, S3_SWDIO, S3_VDD1, S3_VDD10, S3_VDD11, S3_VDD2, S3_VDD3, S3_VDD4, S3_VDD5, S3_VDD6, S3_VDD7, S3_VDD8, S3_VDD9, S3_VDDA, S3_VREF+, S3_VREF-, S3_VSS1, S3_VSS10, S3_VSS11, S3_VSS2, S3_VSS3, S3_VSS4, S3_VSS5, S3_VSS6, S3_VSS7, S3_VSS8, S3_VSS9, S3_VSSA, S4_ADC01, S4_ADC02, S4_ADC03, S4_ADC04, S4_ADC05, S4_ADC06, S4_ADC07, S4_ADC08, S4_ADC09, S4_ADC10, S4_ADC11, S4_ADC12, S4_ADC13, S4_ADC14, S4_ADC15, S4_ADC16, S4_ADC17, S4_ADC18, S4_SPI2_MISO, S4_SPI2_MOSI, S4_SPI2_SCLK, S4_SPI3_MISO, S4_SPI3_MOSI, S4_SPI3_SCK, S4_SWCLK, S4_SWDIO, S4_VDD1, S4_VDD10, S4_VDD11, S4_VDD2, S4_VDD3, S4_VDD4, S4_VDD5, S4_VDD6, S4_VDD7, S4_VDD8, S4_VDD9, S4_VDDA, S4_VREF+, S4_VREF-, S4_VSS1, S4_VSS10, S4_VSS11, S4_VSS2, S4_VSS3, S4_VSS4, S4_VSS5, S4_VSS6, S4_VSS7, S4_VSS8, S4_VSS9, S4_VSSA, SW_RESET, TXN, TXP, W5500_SPI2_MISO, W5500_SPI2_MOSI, W5500_SPI2_SCLK, XI, XO
- net labels removed: DTR, EXT_5V, Earth, JTCK_SWCLK, JTDO, JTMS_SWDIO, RTS, SPI1_MISO, SPI1_MOSI, SPI1_SCK, SPI2_MISO, SPI2_MOSI, SPI2_SCK, USART1_RXD, USART1_TXD, USB_5V, VCC_3.3V, VCC_3V3, VCC_5V
- wire segments 279 -> 527
- no-connect marks 8 -> 346
Other:
- note added: "Back_up_Master"
- note added: "Ethernet"
- note added: "MCU_Slave2"
- note added: "MCU_Slave3"
- note added: "MCU_Slave4"
- note added: "STLink_Master"
- note added: "STLink_Slave"
- note added: "Temperatursensor"
- note removed: "Filter"
- note removed: "ISP"
- note removed: "MCU POWER"
- note removed: "STLink"
- moved on the sheet: BT1, C1, C10, C11, C12, C13, C14, C15, C16, C19, C2, C20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
